Commit message: initial comment

File: urdf/jumping_robot_ry.urdf (robot description, URDF)
Before this commit: robot jumping_robot_ry, 13 links, 12 joints
Links:
- added link base_link
- link ankle_left: mass 0.426454571289873 -> 0.42645; geometry collision mesh filename=package://jumping_robot_ry/meshes/ankle_left.STL; visual mesh filename=package://jumping_robot_ry/meshes/ankle_left.STL
- link ankle_right: mass 0.426454169205949 -> 0.42645; geometry collision mesh filename=package://jumping_robot_ry/meshes/ankle_right.STL; visual mesh filename=package://jumping_robot_ry/meshes/ankle_right.STL
- link arm_left: mass 1.52221564938983 -> 3.5005; geometry collision mesh filename=package://jumping_robot_ry/meshes/arm_left.STL; visual mesh filename=package://jumping_robot_ry/meshes/arm_left.STL
- link arm_right: mass 1.52899552470419 -> 3.5005; geometry collision mesh filename=package://jumping_robot_ry/meshes/arm_right.STL; visual mesh filename=package://jumping_robot_ry/meshes/arm_right.STL
- link calf_left: mass 1.75714585360334 -> 3.3; geometry collision mesh filename=package://jumping_robot_ry/meshes/calf_left.STL; visual mesh filename=package://jumping_robot_ry/meshes/calf_left.STL
- link calf_right: mass 1.77439208129268 -> 3.3; geometry collision mesh filename=package://jumping_robot_ry/meshes/calf_right.STL; visual mesh filename=package://jumping_robot_ry/meshes/calf_right.STL
- link foot_left: mass 1.17881866734593 -> 1.5652; geometry collision mesh filename=package://jumping_robot_ry/meshes/foot_left.STL; visual mesh filename=package://jumping_robot_ry/meshes/foot_left.STL
- link foot_right: mass 1.1788830860114 -> 1.5652; geometry collision mesh filename=package://jumping_robot_ry/meshes/foot_right.STL; visual mesh filename=package://jumping_robot_ry/meshes/foot_right.STL
- link hip_left: mass 2.77226286740998 -> 2.7723; geometry collision mesh filename=package://jumping_robot_ry/meshes/hip_left.STL; visual mesh filename=package://jumping_robot_ry/meshes/hip_left.STL
- link hip_right: mass 2.77194420190797 -> 2.7723; geometry collision mesh filename=package://jumping_robot_ry/meshes/hip_right.STL; visual mesh filename=package://jumping_robot_ry/meshes/hip_right.STL
- link thigh_left: mass 2.24457308468349 -> 4; geometry collision mesh filename=package://jumping_robot_ry/meshes/thigh_left.STL; visual mesh filename=package://jumping_robot_ry/meshes/thigh_left.STL
- link thigh_right: mass 2.24425664830097 -> 4; geometry collision mesh filename=package://jumping_robot_ry/meshes/thigh_right.STL; visual mesh filename=package://jumping_robot_ry/meshes/thigh_right.STL
- link trunk: mass 20.9913292790793 -> 8.19194207079644; geometry collision mesh filename=package://jumping_robot_ry/meshes/trunk.STL; visual mesh filename=package://jumping_robot_ry/meshes/trunk.STL
Joints:
- added joint waist: type fixed, parent base_link, child trunk, origin xyz=0 0 0 rpy=0 0 0
- joint ankle_left_x: limit lower=-3.14 upper=3.14 effort=180 velocity=23.14 -> lower=-3.14 upper=3.14 effort=280 velocity=60.62; origin xyz=0 0 0 rpy=-1.5707963267949 0.0181093582985449 0 -> xyz=0 0 0 rpy=-1.5707963267949 0 0
- joint ankle_left_y: axis 0 0 -1 -> 0 0 1; limit lower=-3.14 upper=3.14 effort=180 velocity=23.14 -> lower=-3.14 upper=3.14 effort=280 velocity=60.62; origin xyz=0.449999999999998 0 0 rpy=0 0 -2.45516141042258E-05 -> xyz=0.45 0 0 rpy=0 0 0
- joint ankle_right_x: limit lower=-3.14 upper=3.14 effort=180 velocity=23.14 -> lower=-3.14 upper=3.14 effort=280 velocity=60.62; origin xyz=0 0 0 rpy=-1.5707963267949 -0.0228520501419932 0 -> xyz=0 0 0 rpy=-1.5707963267949 0 0
- joint ankle_right_y: limit lower=-3.14 upper=3.14 effort=180 velocity=23.14 -> lower=-3.14 upper=3.14 effort=280 velocity=60.62; origin xyz=0.449001113584365 0 0 rpy=0 0 0.00220261619564081 -> xyz=0.449 0 0 rpy=0 0 0
- joint hip_left_x: axis 0.00536591255347294 0 -0.999985603387603 -> 0 0 1; limit lower=-3.14 upper=3.14 effort=180 velocity=23.14 -> lower=-3.14 upper=3.14 effort=280 velocity=60.62; origin xyz=-0.000306223726313573 0.105707340365802 -0.214000000121042 rpy=-2.74895393765495 1.56498843183028 -2.74895989990149 -> xyz=-0.010946 0.083004 -0.223 rpy=0 1.5707963267949 0; type revolute -> fixed
- joint hip_left_y: axis 0.00222221677924413 0 0.999997530873244 -> 0 0 1; limit lower=-3.14 upper=3.14 effort=180 velocity=23.14 -> lower=-3.14 upper=3.14 effort=280 velocity=60.62; origin xyz=0 0 0 rpy=1.57078440237293 0 0 -> xyz=0 0 0 rpy=1.5707963267949 0 0
- joint hip_right_x: limit lower=-3.14 upper=3.14 effort=180 velocity=23.14 -> lower=-3.14 upper=3.14 effort=280 velocity=60.62; origin xyz=-0.000306223726313174 -0.0872016569640492 -0.214000000119806 rpy=0 1.5707963267949 0 -> xyz=-0.010946 -0.091996 -0.223 rpy=0 1.5707963267949 0; type revolute -> fixed
- joint hip_right_y: axis 0.00222221678013116 0 -0.999997530873243 -> 0 0 1; limit lower=-3.14 upper=3.14 effort=180 velocity=23.14 -> lower=-3.14 upper=3.14 effort=280 velocity=60.62; origin xyz=0 0 0 rpy=1.57080825121687 0.00536593827613417 0.0022222506020442 -> xyz=0 0 0 rpy=1.5707963267949 0 0
- joint knee_left: limit lower=-3.14 upper=3.14 effort=180 velocity=23.14 -> lower=-3.14 upper=3.14 effort=280 velocity=60.62; origin xyz=0.45000111110981 0 0 rpy=0 0.00222221714763328 0.00114653302611344 -> xyz=0.45 0 0 rpy=0 0 0
- joint knee_right: axis 0 0 -1 -> 0 0 1; limit lower=-3.14 upper=3.14 effort=180 velocity=23.14 -> lower=-3.14 upper=3.14 effort=280 velocity=60.62; origin xyz=0.45000111111102 0 0 rpy=0 -0.00222221731158092 -0.00108064028281444 -> xyz=0.45 0 0 rpy=0 0 0
- joint shoulder_left: limit lower=-3.14 upper=3.14 effort=180 velocity=23.14 -> lower=-1.7 upper=1.7 effort=280 velocity=60.62; origin xyz=-0.0101075147782717 0.257795843052775 0.165349999885798 rpy=-1.5707963267949 1.56712606042027 3.14159265358979 -> xyz=0.0022528 0.253 0.16485 rpy=-1.5707963267949 1.5707963267949 3.14159265358979
- joint shoulder_right: axis 0 0 -1 -> 0 0 1; limit lower=-3.14 upper=3.14 effort=180 velocity=23.14 -> lower=-1.7 upper=1.7 effort=280 velocity=60.62; origin xyz=-0.0101075147782718 -0.257199156940497 0.165349999885798 rpy=-1.5707963267949 1.56712606042021 3.14159265358979 -> xyz=0.0022528 -0.26199 0.16485 rpy=-1.5707963267949 1.5707963267949 3.14159265358979
